Commit message: add joint dynamics

File: models/urdf/swivel_caster.xacro (robot description, xacro)
@@ -51,4 +51,5 @@
       <origin xyz="-0.2 0 0" rpy="0 0 0"/>
       <limit effort="0" velocity="0"/>
+      <dynamics damping="0.001" friction="0.0001"/>
     </joint>
     <joint name="${prefix}_caster_joint" type="continuous">
@@ -58,4 +59,5 @@
       <origin xyz="-0.03 0 -0.04" rpy="1.52 0 0"/>
       <limit effort="0" velocity="0"/>
+      <dynamics damping="0.001" friction="0.0001"/>
     </joint>
   </xacro:macro>

File: models/urdf/test_robot.urdf.xacro (robot description, xacro)
@@ -62,4 +62,5 @@
     <origin xyz="0 0 0.125" rpy="0 0 0"/>
     <limit effort="0.3" velocity="0.5" lower="-1.52" upper="1.52"/>
+    <dynamics damping="0.01" friction="0.001"/>
   </joint>
   <xacro:include filename="$(find ros_ign_utils)/models/urdf/wheel.xacro"/>

File: models/urdf/wheel.xacro (robot description, xacro)
@@ -29,4 +29,5 @@
       <xacro:insert_block name="origin"/>
       <limit effort="0.5" velocity="1.0"/>
+      <dynamics damping="0.01" friction="0.001"/>
     </joint>
   </xacro:macro>
