Commit message: rename camera.xacro

File: models/urdf/camera_link_macro.xacro (robot description, xacro)
@@ -1,5 +1,5 @@
 <?xml version="1.0"?>
 <robot xmlns:xacro="http://ros.org/wiki/xacro">
-  <xacro:macro name="camera" params="*parent *origin prefix">
+  <xacro:macro name="camera_link_macro" params="*parent *origin prefix">
     <link name="${prefix}_camera_link">
       <origin xyz="0 0 0" rpy="0 0 0"/>
