Commit message: unified xacro macro

File: models/urdf/swivel_caster_link.xacro (robot description, xacro)
@@ -1,5 +1,5 @@
 <?xml version="1.0"?>
 <robot xmlns:xacro="http://ros.org/wiki/xacro">
-  <xacro:macro name="swivel_caster" params="*parent *origin prefix">
+  <xacro:macro name="swivel_caster_link" params="*parent *origin prefix">
     <link name="${prefix}_swivel_link">
       <origin xyz="0 0 0" rpy="0 0 0"/>

File: models/urdf/test_robot.urdf.xacro (robot description, xacro)
@@ -64,22 +64,22 @@
     <dynamics damping="0.01" friction="0.001"/>
   </joint>
-  <xacro:include filename="$(find ros_ign_utils)/models/urdf/wheel.xacro"/>
-  <xacro:wheel prefix="left">
+  <xacro:include filename="$(find ros_ign_utils)/models/urdf/wheel_link.xacro"/>
+  <xacro:wheel_link prefix="left">
     <parent link="lower_body_link"/>
     <origin xyz="0 0.225 -0.03" rpy="1.52 0 0"/>
-  </xacro:wheel>
-  <xacro:wheel prefix="right">
+  </xacro:wheel_link>
+  <xacro:wheel_link prefix="right">
     <parent link="lower_body_link"/>
     <origin xyz="0 -0.225 -0.03" rpy="1.52 0 0"/>
-  </xacro:wheel>
-  <xacro:include filename="$(find ros_ign_utils)/models/urdf/swivel_caster.xacro"/>
-  <xacro:swivel_caster prefix="rear">
+  </xacro:wheel_link>
+  <xacro:include filename="$(find ros_ign_utils)/models/urdf/swivel_caster_link.xacro"/>
+  <xacro:swivel_caster_link prefix="rear">
     <parent link="lower_body_link"/>
     <origin xyz="-0.225 0 0" rpy="0 0 0"/>
-  </xacro:swivel_caster>
-  <xacro:swivel_caster prefix="front">
+  </xacro:swivel_caster_link>
+  <xacro:swivel_caster_link prefix="front">
     <parent link="lower_body_link"/>
     <origin xyz="0.225 0 0" rpy="0 0 0"/>
-  </xacro:swivel_caster>
+  </xacro:swivel_caster_link>
   <xacro:include filename="$(find ros_ign_utils)/models/urdf/camera_link_macro.xacro"/>
   <xacro:camera_link_macro prefix="front">

File: models/urdf/wheel_link.xacro (robot description, xacro)
@@ -1,5 +1,5 @@
 <?xml version="1.0"?>
 <robot xmlns:xacro="http://ros.org/wiki/xacro">
-  <xacro:macro name="wheel" params="*parent *origin prefix">
+  <xacro:macro name="wheel_link" params="*parent *origin prefix">
     <link name="${prefix}_wheel_link">
       <origin xyz="0 0 0" rpy="0 0 0"/>
