Commit message: update  test_bot.urdf.xacro

File: models/urdf/test_robot.urdf.xacro (robot description, xacro)
@@ -78,8 +78,21 @@
     <origin xyz="-0.2 0 0" rpy="0 0 0"/>
   </xacro:swivel_caster>
-  <xacro:include filename="$(find ros_ign_utils)/models/urdf/camera.xacro"/>
-  <xacro:camera prefix="front">
+  <xacro:include filename="$(find ros_ign_utils)/models/urdf/camera_link_macro.xacro"/>
+  <xacro:camera_link_macro prefix="front">
     <parent link="upper_body_link"/>
     <origin xyz="0.28 0 0.1" rpy="0 0 0"/>
-  </xacro:camera>
+  </xacro:camera_link_macro>
+  <xacro:include filename="$(find ros_ign_utils)/models/urdf/imu_link_macro.xacro"/>
+  <xacro:imu_link_macro prefix="upper">
+    <parent link="upper_body_link"/>
+    <origin xyz="0.05 0 0" rpy="0 0 0"/>
+  </xacro:imu_link_macro>
+  <xacro:imu_link_macro prefix="lower">
+    <parent link="lower_body_link"/>
+    <origin xyz="-0.05 0 0" rpy="0 0 0"/>
+  </xacro:imu_link_macro>
+  <gazebo>
+    <plugin filename="ignition-gazebo-joint-state-publisher-system" name="ignition::gazebo::systems::JointStatePublisher">
+    </plugin>
+  </gazebo>
 </robot>

Commit message: update wheels position

File: models/urdf/test_robot.urdf.xacro (robot description, xacro)
@@ -67,14 +67,18 @@
   <xacro:wheel prefix="left">
     <parent link="lower_body_link"/>
-    <origin xyz="0.1 0.225 -0.03" rpy="1.52 0 0"/>
+    <origin xyz="0 0.225 -0.03" rpy="1.52 0 0"/>
   </xacro:wheel>
   <xacro:wheel prefix="right">
     <parent link="lower_body_link"/>
-    <origin xyz="0.1 -0.225 -0.03" rpy="1.52 0 0"/>
+    <origin xyz="0 -0.225 -0.03" rpy="1.52 0 0"/>
   </xacro:wheel>
   <xacro:include filename="$(find ros_ign_utils)/models/urdf/swivel_caster.xacro"/>
   <xacro:swivel_caster prefix="rear">
     <parent link="lower_body_link"/>
-    <origin xyz="-0.2 0 0" rpy="0 0 0"/>
+    <origin xyz="-0.225 0 0" rpy="0 0 0"/>
+  </xacro:swivel_caster>
+  <xacro:swivel_caster prefix="front">
+    <parent link="lower_body_link"/>
+    <origin xyz="0.225 0 0" rpy="0 0 0"/>
   </xacro:swivel_caster>
   <xacro:include filename="$(find ros_ign_utils)/models/urdf/camera_link_macro.xacro"/>

Commit message: add arm_link

File: models/urdf/test_robot.urdf.xacro (robot description, xacro)
@@ -82,4 +82,9 @@
     <origin xyz="0.225 0 0" rpy="0 0 0"/>
   </xacro:swivel_caster_link>
+  <xacro:include filename="$(find ros_ign_utils)/models/urdf/arm_link.xacro"/>
+  <xacro:arm_link prefix="center">
+    <parent link="upper_body_link"/>
+    <origin xyz="0 0 0.1" rpy="0 0 0"/>
+  </xacro:arm_link>
   <xacro:include filename="$(find ros_ign_utils)/models/urdf/camera_link_macro.xacro"/>
   <xacro:camera_link_macro prefix="front">

Commit message: update robot model

File: models/urdf/test_robot.urdf.xacro (robot description, xacro)
@@ -1,4 +1,5 @@
 <?xml version="1.0"?>
 <robot xmlns:xacro="http://ros.org/wiki/xacro" name="test_robot">
+  <xacro:arg name="use_fake_hardware" default="false"/>
   <link name="base_link">
     <origin xyz="0 0 0" rpy="0 0 0"/>
@@ -104,4 +105,36 @@
     <plugin filename="ignition-gazebo-joint-state-publisher-system" name="ignition::gazebo::systems::JointStatePublisher">
     </plugin>
+    <plugin filename="ign_ros2_control-system" name="ign_ros2_control::IgnitionROS2ControlPlugin">
+      <parameters>$(find ros_ign_utils)/config/test_robot_controllers.yaml</parameters>
+      <ros>
+        <remapping>joint_states:=joint_state_broadcaster/joint_states</remapping>
+      </ros>
+    </plugin>
   </gazebo>
+  <ros2_control name="IgnitionSystem" type="system">
+    <hardware>
+      <xacro:if value="$(arg use_fake_hardware)">
+        <plugin>fake_components/GenericSystem</plugin>
+      </xacro:if>
+      <xacro:unless value="$(arg use_fake_hardware)">
+        <plugin>ign_ros2_control/IgnitionSystem</plugin>
+      </xacro:unless>
+    </hardware>
+    <joint name="left_wheel_joint">
+      <command_interface name="velocity">
+        <param name="min">-1</param>
+        <param name="max">1</param>
+      </command_interface>
+      <state_interface name="position"/>
+      <state_interface name="velocity"/>
+    </joint>
+    <joint name="right_wheel_joint">
+      <command_interface name="velocity">
+        <param name="min">-1</param>
+        <param name="max">1</param>
+      </command_interface>
+      <state_interface name="position"/>
+      <state_interface name="velocity"/>
+    </joint>
+  </ros2_control>
 </robot>

Commit message: fix wheel rotate axis

File: models/urdf/test_robot.urdf.xacro (robot description, xacro)
@@ -68,9 +68,9 @@
   <xacro:wheel_link prefix="left">
     <parent link="lower_body_link"/>
-    <origin xyz="0 0.225 -0.03" rpy="1.52 0 0"/>
+    <origin xyz="0 0.225 -0.03" rpy="-1.52 0 0"/>
   </xacro:wheel_link>
   <xacro:wheel_link prefix="right">
     <parent link="lower_body_link"/>
-    <origin xyz="0 -0.225 -0.03" rpy="1.52 0 0"/>
+    <origin xyz="0 -0.225 -0.03" rpy="-1.52 0 0"/>
   </xacro:wheel_link>
   <xacro:include filename="$(find ros_ign_utils)/models/urdf/swivel_caster_link.xacro"/>

Commit message: add joint_trajectory_controller

File: models/urdf/test_robot.urdf.xacro (robot description, xacro)
@@ -137,4 +137,30 @@
       <state_interface name="velocity"/>
     </joint>
+    <joint name="lower_to_upper_joint">
+      <command_interface name="position">
+        <param name="min">-1.57</param>
+        <param name="max">1.57</param>
+      </command_interface>
+      <state_interface name="position"/>
+      <state_interface name="velocity"/>
+    </joint>
+    <joint name="center_lower_arm_joint">
+      <command_interface name="position">
+        <param name="min">-1.57</param>
+        <param name="max">1.57</param>
+      </command_interface>
+      <state_interface name="position"/>
+      <state_interface name="velocity"/>
+      <state_interface name="effort"/>
+    </joint>
+    <joint name="center_upper_arm_joint">
+      <command_interface name="position">
+        <param name="min">-1.57</param>
+        <param name="max">1.57</param>
+      </command_interface>
+      <state_interface name="position"/>
+      <state_interface name="velocity"/>
+      <state_interface name="effort"/>
+    </joint>
   </ros2_control>
 </robot>
