Commit message: add forcetorque sensor and navsat sensor

File: models/urdf/test_robot/test_robot.urdf.xacro (robot description, xacro)
@@ -102,4 +102,9 @@
     <origin xyz="-0.05 0 0" rpy="0 0 0"/>
   </xacro:imu_link_macro>
+  <xacro:include filename="navsat_link_macro.xacro"/>
+  <xacro:navsat_link_macro prefix="upper">
+    <parent link="upper_body_link"/>
+    <origin xyz="0.1 0 0.05" rpy="0 0 0"/>
+  </xacro:navsat_link_macro>
   <gazebo>
     <plugin filename="ignition-gazebo-joint-state-publisher-system" name="ignition::gazebo::systems::JointStatePublisher">

File: models/urdf/test_robot/wheel_link.xacro (robot description, xacro)
@@ -31,4 +31,14 @@
       <dynamics damping="0.01" friction="0.001"/>
     </joint>
+    <gazebo reference="${prefix}_wheel_joint">
+      <sensor name="${prefix}_wheel_force_torque_sensor" type="force_torque">
+        <always_on>true</always_on>
+        <update_rate>10</update_rate>
+      </sensor>
+    </gazebo>
   </xacro:macro>
+  <gazebo>
+    <plugin filename="ignition-gazebo-forcetorque-system" name="ignition::gazebo::systems::ForceTorque">
+    </plugin>
+  </gazebo>
 </robot>

Commit message: add laser scan sensor

File: models/urdf/test_robot/test_robot.urdf.xacro (robot description, xacro)
@@ -86,5 +86,5 @@
   <xacro:arm_link prefix="center">
     <parent link="upper_body_link"/>
-    <origin xyz="0 0 0.1" rpy="0 0 0"/>
+    <origin xyz="0 0 0.2" rpy="0 0 0"/>
   </xacro:arm_link>
   <xacro:include filename="camera_link_macro.xacro"/>
@@ -107,4 +107,9 @@
     <origin xyz="0.1 0 0.05" rpy="0 0 0"/>
   </xacro:navsat_link_macro>
+  <xacro:include filename="scan_link_macro.xacro"/>
+  <xacro:scan_link_macro prefix="upper">
+    <parent link="upper_body_link"/>
+    <origin xyz="0 0 0.125" rpy="0 0 0"/>
+  </xacro:scan_link_macro>
   <gazebo>
     <plugin filename="ignition-gazebo-joint-state-publisher-system" name="ignition::gazebo::systems::JointStatePublisher">
