Commit message: Fix passive force joint

File: models/urdf/test_robot/swivel_caster_link.xacro (robot description, xacro)
@@ -50,6 +50,6 @@
       <xacro:insert_block name="origin"/>
       <origin xyz="-0.2 0 0" rpy="0 0 0"/>
-      <limit effort="0" velocity="0"/>
-      <dynamics damping="0.001" friction="0.0001"/>
+      <limit effort="10" velocity="10"/>
+      <dynamics damping="0.0" friction="0.0"/>
     </joint>
     <joint name="${prefix}_caster_joint" type="continuous">
@@ -58,6 +58,6 @@
       <axis xyz="0 0 1"/>
       <origin xyz="-0.03 0 -0.04" rpy="1.52 0 0"/>
-      <limit effort="0" velocity="0"/>
-      <dynamics damping="0.001" friction="0.0001"/>
+      <limit effort="10" velocity="10"/>
+      <dynamics damping="0.0" friction="0.0"/>
     </joint>
   </xacro:macro>

File: models/urdf/test_robot/test_robot.urdf.xacro (robot description, xacro)
@@ -151,6 +151,6 @@
     <joint name="left_wheel_joint">
       <command_interface name="velocity">
-        <param name="min">-1</param>
-        <param name="max">1</param>
+        <param name="min">-5</param>
+        <param name="max">5</param>
       </command_interface>
       <state_interface name="position"/>
@@ -159,6 +159,6 @@
     <joint name="right_wheel_joint">
       <command_interface name="velocity">
-        <param name="min">-1</param>
-        <param name="max">1</param>
+        <param name="min">-5</param>
+        <param name="max">5</param>
       </command_interface>
       <state_interface name="position"/>

File: models/urdf/test_robot/wheel_link.xacro (robot description, xacro)
@@ -28,5 +28,5 @@
       <axis xyz="0 0 1"/>
       <xacro:insert_block name="origin"/>
-      <limit effort="0.5" velocity="1.0"/>
+      <limit effort="1.0" velocity="4.0"/>
       <dynamics damping="0.01" friction="0.001"/>
     </joint>
